Commit message: launched model in gazebo

File: src/description/urdf/argus.urdf.xacro (robot description, xacro)
@@ -1,4 +1,8 @@
 <?xml version="1.0"?>
 <robot name="argus" xmlns:xacro="http://www.ros.org/wiki/xacro">
+  <!-- Add a Gazebo reference for the blue color -->
+  <gazebo reference="base_link">
+    <material>Gazebo/Blue</material>
+  </gazebo>
   <link name="base_link">
     <visual>
@@ -15,4 +19,13 @@
       </geometry>
     </collision>
+    <!-- CRITICAL: Added inertial properties for the physics simulation -->
+    <inertial>
+      <!-- Mass in kilograms -->
+      <mass value="5.0"/>
+      <!-- Inertia matrix for a box -->
+      <inertia ixx="0.01" ixy="0.0" ixz="0.0"
+               iyy="0.01" iyz="0.0"
+               izz="0.01"/>
+    </inertial>
   </link>
 </robot>

Commit message: error in controlling bot

File: src/description/urdf/argus.urdf.xacro (robot description, xacro)
@@ -1,8 +1,41 @@
 <?xml version="1.0"?>
 <robot name="argus" xmlns:xacro="http://www.ros.org/wiki/xacro">
-  <!-- Add a Gazebo reference for the blue color -->
-  <gazebo reference="base_link">
-    <material>Gazebo/Blue</material>
-  </gazebo>
+  <material name="blue">
+    <color rgba="0.0 0.0 0.8 1.0"/>
+  </material>
+  <material name="grey">
+    <color rgba="0.5 0.5 0.5 1.0"/>
+  </material>
+  <xacro:property name="wheel_radius" value="0.05" />
+  <xacro:property name="wheel_height" value="0.04" />
+  <xacro:property name="wheel_mass" value="0.5" />
+  <xacro:macro name="wheel" params="prefix parent">
+    <link name="${prefix}_wheel_link">
+      <visual>
+        <geometry>
+          <cylinder radius="${wheel_radius}" length="${wheel_height}"/>
+        </geometry>
+        <material name="grey"/>
+      </visual>
+      <collision>
+        <geometry>
+          <cylinder radius="${wheel_radius}" length="${wheel_height}"/>
+        </geometry>
+      </collision>
+      <inertial>
+        <mass value="${wheel_mass}"/>
+        <inertia ixx="0.001" ixy="0.0" ixz="0.0" iyy="0.001" iyz="0.0" izz="0.001"/>
+      </inertial>
+    </link>
+    <joint name="${prefix}_wheel_joint" type="continuous">
+      <parent link="${parent}"/>
+      <child link="${prefix}_wheel_link"/>
+      <origin xyz="0 0 0" rpy="-1.5707 0 0"/>
+      <axis xyz="0 0 1"/>
+    </joint>
+    <gazebo reference="${prefix}_wheel_link">
+      <material>Gazebo/Grey</material>
+    </gazebo>
+  </xacro:macro>
   <link name="base_link">
     <visual>
@@ -10,7 +43,5 @@
         <box size="0.5 0.3 0.1"/>
       </geometry>
-      <material name="blue">
-        <color rgba="0.0 0.0 0.8 1.0"/>
-      </material>
+      <material name="blue"/>
     </visual>
     <collision>
@@ -19,13 +50,45 @@
       </geometry>
     </collision>
-    <!-- CRITICAL: Added inertial properties for the physics simulation -->
     <inertial>
-      <!-- Mass in kilograms -->
       <mass value="5.0"/>
-      <!-- Inertia matrix for a box -->
-      <inertia ixx="0.01" ixy="0.0" ixz="0.0"
-               iyy="0.01" iyz="0.0"
-               izz="0.01"/>
+      <inertia ixx="0.01" ixy="0.0" ixz="0.0" iyy="0.01" iyz="0.0" izz="0.01"/>
     </inertial>
   </link>
+  <gazebo reference="base_link">
+    <material>Gazebo/Blue</material>
+  </gazebo>
+  <link name="front_left_mount"/>
+  <link name="front_right_mount"/>
+  <link name="rear_left_mount"/>
+  <link name="rear_right_mount"/>
+  <joint name="front_left_mount_joint" type="fixed"><parent link="base_link"/><child link="front_left_mount"/><origin xyz="0.15 0.17 0"/></joint>
+  <joint name="front_right_mount_joint" type="fixed"><parent link="base_link"/><child link="front_right_mount"/><origin xyz="0.15 -0.17 0"/></joint>
+  <joint name="rear_left_mount_joint" type="fixed"><parent link="base_link"/><child link="rear_left_mount"/><origin xyz="-0.15 0.17 0"/></joint>
+  <joint name="rear_right_mount_joint" type="fixed"><parent link="base_link"/><child link="rear_right_mount"/><origin xyz="-0.15 -0.17 0"/></joint>
+  <xacro:wheel prefix="front_left" parent="front_left_mount"/>
+  <xacro:wheel prefix="front_right" parent="front_right_mount"/>
+  <xacro:wheel prefix="rear_left" parent="rear_left_mount"/>
+  <xacro:wheel prefix="rear_right" parent="rear_right_mount"/>
+  <gazebo>
+    <plugin name="diff_drive_controller" filename="libgazebo_ros_diff_drive.so">
+      <ros>
+        <namespace>/argus</namespace>
+      </ros>
+      <left_joint>front_left_wheel_joint</left_joint>
+      <left_joint>rear_left_wheel_joint</left_joint>
+      <right_joint>front_right_wheel_joint</right_joint>
+      <right_joint>rear_right_wheel_joint</right_joint>
+      <wheel_separation>0.34</wheel_separation>
+      <wheel_diameter>0.1</wheel_diameter>
+      <max_wheel_torque>20</max_wheel_torque>
+      <max_wheel_acceleration>1.0</max_wheel_acceleration>
+      <command_topic>cmd_vel</command_topic>
+      <odometry_topic>odom</odometry_topic>
+      <odometry_frame>odom</odometry_frame>
+      <robot_base_frame>base_link</robot_base_frame>
+      <publish_odom>true</publish_odom>
+      <publish_odom_tf>true</publish_odom_tf>
+      <publish_wheel_tf>false</publish_wheel_tf>
+    </plugin>
+  </gazebo>
 </robot>

Commit message: setting up rviz

File: src/description/urdf/argus.urdf.xacro (robot description, xacro)
@@ -1,4 +1,5 @@
 <?xml version="1.0"?>
 <robot name="argus" xmlns:xacro="http://www.ros.org/wiki/xacro">
+  <!-- ############ MATERIALS ############ -->
   <material name="blue">
     <color rgba="0.0 0.0 0.8 1.0"/>
@@ -7,4 +8,5 @@
     <color rgba="0.5 0.5 0.5 1.0"/>
   </material>
+  <!-- ############ WHEEL MACRO ############ -->
   <xacro:property name="wheel_radius" value="0.05" />
   <xacro:property name="wheel_height" value="0.04" />
@@ -38,4 +40,5 @@
     </gazebo>
   </xacro:macro>
+  <!-- ############ ROBOT BODY (BASE LINK) ############ -->
   <link name="base_link">
     <visual>
@@ -58,4 +61,5 @@
     <material>Gazebo/Blue</material>
   </gazebo>
+  <!-- ############ WHEEL MOUNTS ############ -->
   <link name="front_left_mount"/>
   <link name="front_right_mount"/>
@@ -66,29 +70,82 @@
   <joint name="rear_left_mount_joint" type="fixed"><parent link="base_link"/><child link="rear_left_mount"/><origin xyz="-0.15 0.17 0"/></joint>
   <joint name="rear_right_mount_joint" type="fixed"><parent link="base_link"/><child link="rear_right_mount"/><origin xyz="-0.15 -0.17 0"/></joint>
+  <!-- Attach wheels using the macro -->
   <xacro:wheel prefix="front_left" parent="front_left_mount"/>
   <xacro:wheel prefix="front_right" parent="front_right_mount"/>
   <xacro:wheel prefix="rear_left" parent="rear_left_mount"/>
   <xacro:wheel prefix="rear_right" parent="rear_right_mount"/>
+  <!-- ############ LIDAR SENSOR ############ -->
+  <link name="laser_link">
+    <visual>
+      <geometry>
+        <cylinder radius="0.03" length="0.05"/>
+      </geometry>
+      <material name="grey"/>
+    </visual>
+    <collision>
+      <geometry>
+        <cylinder radius="0.03" length="0.05"/>
+      </geometry>
+    </collision>
+    <inertial>
+      <mass value="0.1"/>
+      <inertia ixx="0.0001" ixy="0.0" ixz="0.0" iyy="0.0001" iyz="0.0" izz="0.0001"/>
+    </inertial>
+  </link>
+  <joint name="laser_joint" type="fixed">
+    <parent link="base_link"/>
+    <child link="laser_link"/>
+    <origin xyz="0.2 0 0.1" rpy="0 0 0"/>
+  </joint>
+  <!-- ############ GAZEBO PLUGINS ############ -->
   <gazebo>
+    <!-- Differential Drive Controller -->
     <plugin name="diff_drive_controller" filename="libgazebo_ros_diff_drive.so">
-      <ros>
-        <namespace>/argus</namespace>
-      </ros>
-      <left_joint>front_left_wheel_joint</left_joint>
-      <left_joint>rear_left_wheel_joint</left_joint>
-      <right_joint>front_right_wheel_joint</right_joint>
-      <right_joint>rear_right_wheel_joint</right_joint>
-      <wheel_separation>0.34</wheel_separation>
-      <wheel_diameter>0.1</wheel_diameter>
-      <max_wheel_torque>20</max_wheel_torque>
-      <max_wheel_acceleration>1.0</max_wheel_acceleration>
-      <command_topic>cmd_vel</command_topic>
-      <odometry_topic>odom</odometry_topic>
-      <odometry_frame>odom</odometry_frame>
-      <robot_base_frame>base_link</robot_base_frame>
-      <publish_odom>true</publish_odom>
-      <publish_odom_tf>true</publish_odom_tf>
-      <publish_wheel_tf>false</publish_wheel_tf>
+      <rosNamespace>/argus</rosNamespace>
+      <commandTopic>cmd_vel</commandTopic>
+      <odometryTopic>odom</odometryTopic>
+      <odometryFrame>odom</odometryFrame>
+      <robotBaseFrame>base_link</robotBaseFrame>
+      <!-- This is the critical line that fixes the RobotModel error in RViz -->
+      <publishWheelJointState>true</publishWheelJointState>
+      <leftJoint>front_left_wheel_joint</leftJoint>
+      <leftJoint>rear_left_wheel_joint</leftJoint>
+      <rightJoint>front_right_wheel_joint</rightJoint>
+      <rightJoint>rear_right_wheel_joint</rightJoint>
+      <wheelSeparation>0.34</wheelSeparation>
+      <wheelDiameter>0.1</wheelDiameter>
+      <maxWheelTorque>20</maxWheelTorque>
+      <maxWheelAcceleration>1.0</maxWheelAcceleration>
+      <publishOdom>true</publishOdom>
+      <publishOdomTF>true</publishOdomTF>
+      <publishWheelTF>false</publishWheelTF>
     </plugin>
   </gazebo>
+  <gazebo reference="laser_link">
+    <!-- LiDAR Sensor Plugin -->
+    <sensor type="ray" name="head_hokuyo_sensor">
+      <pose>0 0 0 0 0 0</pose>
+      <visualize>true</visualize>
+      <update_rate>20</update_rate>
+      <ray>
+        <scan>
+          <horizontal>
+            <samples>720</samples>
+            <resolution>1</resolution>
+            <min_angle>-1.5708</min_angle>
+            <max_angle>1.5708</max_angle>
+          </horizontal>
+        </scan>
+        <range>
+          <min>0.10</min>
+          <max>10.0</max>
+          <resolution>0.01</resolution>
+        </range>
+      </ray>
+      <plugin name="gazebo_ros_head_hokuyo_controller" filename="libgazebo_ros_laser.so">
+        <topicName>/argus/scan</topicName>
+        <frameName>laser_link</frameName>
+      </plugin>
+    </sensor>
+  </gazebo>
 </robot>

Commit message: changed model colors

File: src/description/urdf/argus.urdf.xacro (robot description, xacro)
@@ -7,4 +7,28 @@
   <material name="grey">
     <color rgba="0.5 0.5 0.5 1.0"/>
+  </material>
+  <material name="red">
+    <color rgba="1.0 0.0 0.0 1.0"/>
+  </material>
+    <material name="translucent_red">
+    <color rgba="0.8 0.0 0.0 0.5"/>
+  </material>
+  <material name="translucent_blue">
+    <color rgba="0.0 0.0 0.8 0.5"/>
+  </material>
+    <material name="gold">
+    <color rgba="0.83 0.69 0.22 1.0"/>
+  </material>
+  <material name="silver">
+    <color rgba="0.75 0.75 0.75 1.0"/>
+  </material>
+  <material name="bronze">
+    <color rgba="0.8 0.5 0.2 1.0"/>
+  </material>
+  <material name="steel_blue">
+    <color rgba="0.27 0.51 0.71 1.0"/>
+  </material>
+  <material name="chassis_color">
+    <color rgba="0.2 0.2 0.2 1.0"/>
   </material>
   <!-- ############ WHEEL MACRO ############ -->
@@ -46,5 +70,5 @@
         <box size="0.5 0.3 0.1"/>
       </geometry>
-      <material name="blue"/>
+      <material name="chassis_color"/>
     </visual>
     <collision>
@@ -59,5 +83,9 @@
   </link>
   <gazebo reference="base_link">
-    <material>Gazebo/Blue</material>
+    <material>
+      <ambient>0.2 0.2 0.2 1.0</ambient>
+      <diffuse>0.2 0.2 0.2 1.0</diffuse>
+      <specular>0.2 0.2 0.2 1.0</specular>
+    </material>
   </gazebo>
   <!-- ############ WHEEL MOUNTS ############ -->
@@ -81,5 +109,5 @@
         <cylinder radius="0.03" length="0.05"/>
       </geometry>
-      <material name="grey"/>
+      <material name="translucent_red"/>
     </visual>
     <collision>

Commit message: improvements

File: src/description/urdf/argus.urdf.xacro (robot description, xacro)
@@ -1,40 +1,22 @@
 <?xml version="1.0"?>
 <robot name="argus" xmlns:xacro="http://www.ros.org/wiki/xacro">
+  <!-- ############ GLOBAL PREFIX ############ -->
+  <xacro:property name="prefix" value=""/>
   <!-- ############ MATERIALS ############ -->
-  <material name="blue">
-    <color rgba="0.0 0.0 0.8 1.0"/>
-  </material>
-  <material name="grey">
-    <color rgba="0.5 0.5 0.5 1.0"/>
-  </material>
-  <material name="red">
-    <color rgba="1.0 0.0 0.0 1.0"/>
-  </material>
-    <material name="translucent_red">
-    <color rgba="0.8 0.0 0.0 0.5"/>
-  </material>
-  <material name="translucent_blue">
-    <color rgba="0.0 0.0 0.8 0.5"/>
-  </material>
-    <material name="gold">
-    <color rgba="0.83 0.69 0.22 1.0"/>
-  </material>
-  <material name="silver">
-    <color rgba="0.75 0.75 0.75 1.0"/>
-  </material>
-  <material name="bronze">
-    <color rgba="0.8 0.5 0.2 1.0"/>
-  </material>
-  <material name="steel_blue">
-    <color rgba="0.27 0.51 0.71 1.0"/>
-  </material>
-  <material name="chassis_color">
-    <color rgba="0.2 0.2 0.2 1.0"/>
-  </material>
+  <material name="blue"><color rgba="0 0 0.8 1.0"/></material>
+  <material name="grey"><color rgba="0.5 0.5 0.5 1.0"/></material>
+  <material name="red"><color rgba="1 0 0 1.0"/></material>
+  <material name="translucent_red"><color rgba="0.8 0 0 0.5"/></material>
+  <material name="translucent_blue"><color rgba="0 0 0.8 0.5"/></material>
+  <material name="gold"><color rgba="0.83 0.69 0.22 1.0"/></material>
+  <material name="silver"><color rgba="0.75 0.75 0.75 1.0"/></material>
+  <material name="bronze"><color rgba="0.8 0.5 0.2 1.0"/></material>
+  <material name="steel_blue"><color rgba="0.27 0.51 0.71 1.0"/></material>
+  <material name="chassis_color"><color rgba="0.2 0.2 0.2 1.0"/></material>
   <!-- ############ WHEEL MACRO ############ -->
-  <xacro:property name="wheel_radius" value="0.05" />
-  <xacro:property name="wheel_height" value="0.04" />
-  <xacro:property name="wheel_mass" value="0.5" />
-  <xacro:macro name="wheel" params="prefix parent">
+  <xacro:property name="wheel_radius" value="0.05"/>
+  <xacro:property name="wheel_height" value="0.04"/>
+  <xacro:property name="wheel_mass" value="0.5"/>
+  <xacro:macro name="wheel" params="prefix parent=''">
     <link name="${prefix}_wheel_link">
       <visual>
@@ -51,5 +33,5 @@
       <inertial>
         <mass value="${wheel_mass}"/>
-        <inertia ixx="0.001" ixy="0.0" ixz="0.0" iyy="0.001" iyz="0.0" izz="0.001"/>
+        <inertia ixx="0.001" ixy="0" ixz="0" iyy="0.001" iyz="0" izz="0.001"/>
       </inertial>
     </link>
@@ -57,35 +39,32 @@
       <parent link="${parent}"/>
       <child link="${prefix}_wheel_link"/>
-      <origin xyz="0 0 0" rpy="-1.5707 0 0"/>
-      <axis xyz="0 0 1"/>
+      <origin xyz="0 0 -0.05" rpy="1.5707 0 0"/>
+      <axis xyz="0 1 0"/>
     </joint>
     <gazebo reference="${prefix}_wheel_link">
-      <material>Gazebo/Grey</material>
+        <material>Gazebo/Grey</material>
+        <mu1>1.0</mu1>
+        <mu2>1.0</mu2>
+        <kp>100000</kp>
+        <kd>1</kd>
     </gazebo>
   </xacro:macro>
-  <!-- ############ ROBOT BODY (BASE LINK) ############ -->
+  <!-- ############ BASE LINK ############ -->
   <link name="base_link">
     <visual>
-      <geometry>
-        <box size="0.5 0.3 0.1"/>
-      </geometry>
+      <geometry><box size="0.5 0.3 0.1"/></geometry>
       <material name="chassis_color"/>
     </visual>
     <collision>
-      <geometry>
-        <box size="0.5 0.3 0.1"/>
-      </geometry>
+      <geometry><box size="0.5 0.3 0.1"/></geometry>
     </collision>
     <inertial>
       <mass value="5.0"/>
-      <inertia ixx="0.01" ixy="0.0" ixz="0.0" iyy="0.01" iyz="0.0" izz="0.01"/>
+      <inertia ixx="0.1" ixy="0" ixz="0" iyy="0.2" iyz="0" izz="0.15"/>
     </inertial>
   </link>
   <gazebo reference="base_link">
-    <material>
-      <ambient>0.2 0.2 0.2 1.0</ambient>
-      <diffuse>0.2 0.2 0.2 1.0</diffuse>
-      <specular>0.2 0.2 0.2 1.0</specular>
-    </material>
+  <gravity>true</gravity>
+    <material><ambient>0.2 0.2 0.2 1</ambient><diffuse>0.2 0.2 0.2 1</diffuse><specular>0.2 0.2 0.2 1</specular></material>
   </gazebo>
   <!-- ############ WHEEL MOUNTS ############ -->
@@ -94,80 +73,104 @@
   <link name="rear_left_mount"/>
   <link name="rear_right_mount"/>
-  <joint name="front_left_mount_joint" type="fixed"><parent link="base_link"/><child link="front_left_mount"/><origin xyz="0.15 0.17 0"/></joint>
-  <joint name="front_right_mount_joint" type="fixed"><parent link="base_link"/><child link="front_right_mount"/><origin xyz="0.15 -0.17 0"/></joint>
-  <joint name="rear_left_mount_joint" type="fixed"><parent link="base_link"/><child link="rear_left_mount"/><origin xyz="-0.15 0.17 0"/></joint>
-  <joint name="rear_right_mount_joint" type="fixed"><parent link="base_link"/><child link="rear_right_mount"/><origin xyz="-0.15 -0.17 0"/></joint>
-  <!-- Attach wheels using the macro -->
+  <joint name="front_left_mount_joint" type="fixed">
+    <parent link="base_link"/><child link="front_left_mount"/>
+    <origin xyz="0.15 0.17 0"/>
+    <geometry>
+      <box size="0.02 0.02 0.02"/>
+    </geometry>
+  </joint>
+  <joint name="front_right_mount_joint" type="fixed">
+    <parent link="base_link"/><child link="front_right_mount"/>
+    <origin xyz="0.15 -0.17 0"/>
+    <geometry>
+      <box size="0.02 0.02 0.02"/>
+    </geometry>
+  </joint>
+  <joint name="rear_left_mount_joint" type="fixed">
+    <parent link="base_link"/><child link="rear_left_mount"/>
+    <origin xyz="-0.15 0.17 0"/>
+    <geometry>
+      <box size="0.02 0.02 0.02"/>
+    </geometry>
+  </joint>
+  <joint name="rear_right_mount_joint" type="fixed">
+    <parent link="base_link"/><child link="rear_right_mount"/>
+    <origin xyz="-0.15 -0.17 0"/>
+    <geometry>
+      <box size="0.02 0.02 0.02"/>
+    </geometry>
+  </joint>
+  <!-- ############ ATTACH WHEELS ############ -->
   <xacro:wheel prefix="front_left" parent="front_left_mount"/>
   <xacro:wheel prefix="front_right" parent="front_right_mount"/>
   <xacro:wheel prefix="rear_left" parent="rear_left_mount"/>
   <xacro:wheel prefix="rear_right" parent="rear_right_mount"/>
-  <!-- ############ LIDAR SENSOR ############ -->
+  <!-- ############ GAZEBO SKID STEER PLUGIN ############ -->
+  <gazebo>
+    <plugin name="skid_steer_drive_controller" filename="libgazebo_ros_skid_steer_drive.so">
+      <updateRate>25.0</updateRate>
+      <broadcastTF>true</broadcastTF>
+      <leftFrontJoint>front_left_wheel_joint</leftFrontJoint>
+      <rightFrontJoint>front_right_wheel_joint</rightFrontJoint>
+      <leftRearJoint>rear_left_wheel_joint</leftRearJoint>
+      <rightRearJoint>rear_right_wheel_joint</rightRearJoint>
+      <wheelSeparation>0.34</wheelSeparation>
+      <wheelDiameter>0.1</wheelDiameter>
+      <robotBaseFrame>base_link</robotBaseFrame>
+      <commandTopic>cmd_vel</commandTopic>
+      <odometryTopic>odom</odometryTopic>
+      <odometryFrame>odom</odometryFrame>
+      <torque>20</torque>
+    </plugin>
+  </gazebo>
+  <!-- ############ LIDAR PLUGIN ############ -->
   <link name="laser_link">
-    <visual>
-      <geometry>
-        <cylinder radius="0.03" length="0.05"/>
-      </geometry>
-      <material name="translucent_red"/>
-    </visual>
-    <collision>
-      <geometry>
-        <cylinder radius="0.03" length="0.05"/>
-      </geometry>
-    </collision>
-    <inertial>
-      <mass value="0.1"/>
-      <inertia ixx="0.0001" ixy="0.0" ixz="0.0" iyy="0.0001" iyz="0.0" izz="0.0001"/>
-    </inertial>
-  </link>
-  <joint name="laser_joint" type="fixed">
-    <parent link="base_link"/>
-    <child link="laser_link"/>
-    <origin xyz="0.2 0 0.1" rpy="0 0 0"/>
-  </joint>
-  <!-- ############ GAZEBO PLUGINS ############ -->
-<gazebo>
-  <plugin name="skid_steer_drive_controller" filename="libgazebo_ros_skid_steer_drive.so">
-    <updateRate>25.0</updateRate>
-    <broadcastTF>true</broadcastTF>
-    <leftFrontJoint>front_left_wheel_joint</leftFrontJoint>
-    <rightFrontJoint>front_right_wheel_joint</rightFrontJoint>
-    <leftRearJoint>rear_left_wheel_joint</leftRearJoint>
-    <rightRearJoint>rear_right_wheel_joint</rightRearJoint>
-    <wheelSeparation>0.34</wheelSeparation>
-    <wheelDiameter>0.1</wheelDiameter>
-    <robotBaseFrame>base_link</robotBaseFrame>
-    <commandTopic>cmd_vel</commandTopic>
-    <odometryTopic>odom</odometryTopic>
-    <odometryFrame>odom</odometryFrame>
-    <torque>20</torque>
-  </plugin>
+  <visual>
+    <geometry><cylinder radius="0.03" length="0.05"/></geometry>
+    <material name="translucent_red"/>
+  </visual>
+  <collision>
+    <geometry><cylinder radius="0.03" length="0.05"/></geometry>
+  </collision>
+  <inertial>
+    <mass value="0.1"/>
+    <inertia ixx="0.0001" ixy="0" ixz="0" iyy="0.0001" iyz="0" izz="0.0001"/>
+  </inertial>
+</link>
+<joint name="laser_joint" type="fixed">
+  <parent link="base_link"/>
+  <child link="laser_link"/>
+  <origin xyz="0 0 0.2" rpy="0 0 0"/>
+</joint>
+<gazebo reference="laser_link">
+  <sensor type="ray" name="head_hokuyo_sensor">
+    <pose>0 0 0 0 0 0</pose>
+    <visualize>true</visualize>
+    <update_rate>20</update_rate>
+    <ray>
+      <scan>
+        <horizontal>
+          <samples>720</samples>
+          <resolution>1</resolution>
+          <min_angle>-1.570796</min_angle>
+          <max_angle>1.570796</max_angle>
+        </horizontal>
+      </scan>
+      <range>
+        <min>0.10</min>
+        <max>10.0</max>
+        <resolution>0.01</resolution>
+      </range>
+      <noise>
+        <type>gaussian</type>
+        <mean>0.0</mean>
+        <stddev>0.01</stddev>
+      </noise>
+    </ray>
+    <plugin name="gazebo_ros_head_hokuyo_controller" filename="libgazebo_ros_laser.so">
+      <topicName>/scan</topicName>
+      <frameName>laser_link</frameName>
+    </plugin>
+  </sensor>
 </gazebo>
-  <gazebo reference="laser_link">
-    <!-- LiDAR Sensor Plugin -->
-    <sensor type="ray" name="head_hokuyo_sensor">
-      <pose>0 0 0 0 0 0</pose>
-      <visualize>true</visualize>
-      <update_rate>20</update_rate>
-      <ray>
-        <scan>
-          <horizontal>
-            <samples>720</samples>
-            <resolution>1</resolution>
-            <min_angle>-1.5708</min_angle>
-            <max_angle>1.5708</max_angle>
-          </horizontal>
-        </scan>
-        <range>
-          <min>0.10</min>
-          <max>10.0</max>
-          <resolution>0.01</resolution>
-        </range>
-      </ray>
-      <plugin name="gazebo_ros_head_hokuyo_controller" filename="libgazebo_ros_laser.so">
-        <topicName>/argus/scan</topicName>
-        <frameName>laser_link</frameName>
-      </plugin>
-    </sensor>
-  </gazebo>
 </robot>
